File: p18pyro.X/pyro18.sch (EAGLE design)
At the start: 25 parts, among them U1 TPIC6B595PTH, U2 TPIC6B595PTH, X1 332-10, X2 332-10, X3 332-10, X4 332-10, X5 22-23-2041, X6 out2 pins, X7 22-23-2021

Commit message: updates
Parts:
- X1: value 332-10 -> port c
- X2: value 332-10 -> analog I/O bus
- X3: value 332-10 -> port a
Changed lines of the file:
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@@
 <part name="U1" library="SparkFun-DigitalIC" deviceset="TPIC6B595" device="PTH"/>
 <part name="U2" library="SparkFun-DigitalIC" deviceset="TPIC6B595" device="PTH"/>
-<part name="X1" library="con-garry" deviceset="332-10" device=""/>
-<part name="X2" library="con-garry" deviceset="332-10" device=""/>
-<part name="X3" library="con-garry" deviceset="332-10" device=""/>
+<part name="X1" library="con-garry" deviceset="332-10" device="" value="port c"/>
+<part name="X2" library="con-garry" deviceset="332-10" device="" value="analog I/O bus"/>
+<part name="X3" library="con-garry" deviceset="332-10" device="" value="port a"/>
 <part name="X4" library="con-garry" deviceset="332-10" device=""/>
 <part name="DIS1" library="display-hp" deviceset="HP5082" device=""/>
