File: p18pyro.X/pyro18.brd (EAGLE design)
At the start: 160 x 100 mm, 17 parts, among them U1 TPIC6B595PTH, U2 TPIC6B595PTH, X1 332-10, X2 332-10, X3 332-10, X4 332-10, X5 22-23-2041, X7 22-23-2021

Commit message: updates
Parts:
- added C1, C2, C3, C4, C5, C6: (no value), rcl:C0805
- added LED1: (no value), led:LED3MM
- added R6: (no value), resistor:0207/2V
- moved U$1 1.27 mm to (50.8, 61.0)
- moved U$2 1.27 mm to (41.9, 61.0)
Connections:
- new net N$25: U1.5, X5.2
- new net N$28: U1.6, X5.3
- new net N$29: U1.14, X6.2
- new net N$30: U1.7, X6.1
- new net N$31: U1.15, X6.3
- new net N$32: U1.16, X6.4
- new net N$33: U2.4, X6.5
- new net N$34: U2.5, X6.6
- new net N$35: C6.1, LED1.A, R6.1
- new net N$8: U1.4, X5.1
- net GND: now also C1.2, C2.2, C3.1, C4.1, C5.2, C6.2, LED1.K
- net VCC: now also C3.2, C4.2, C5.1
- net VDD: now also C1.1, C2.1, R6.2
Routing:
- net GND: track 166.4 -> 256.7 mm
- net N$35: track 0.00 -> 84.7 mm
- net VDD: track 52.9 -> 129.6 mm
- net N$34: track 0.00 -> 55.5 mm
- net N$33: track 0.00 -> 50.1 mm
- net N$13: track 29.4 -> 64.2 mm, vias 2 -> 3
- net N$16: track 54.3 -> 85.8 mm
- net N$3: track 58.4 -> 28.1 mm
- net VCC: track 91.2 -> 121.0 mm
- net N$32: track 0.00 -> 27.6 mm
- net N$31: track 0.00 -> 24.8 mm
- net N$29: track 0.00 -> 23.2 mm
- net N$27: track 15.9 -> 36.9 mm
- net N$28: track 0.00 -> 20.7 mm
- net N$4: track 51.4 -> 33.2 mm
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Other:
- board size 160 x 100 mm -> 74.9 x 46.7 mm

Commit message: update
Parts:
- C1, C2, C3, C4, C5: value (none) -> 0.1
- C6: value (none) -> 22uf
- LED1: value (none) -> red
- R1: value (none) -> 662
- R2, R3, R4, R5, R6: value (none) -> 1k
- X6: value (none) -> out2 pins
Connections:
- removed net N$11: X7.1
- removed net N$5: U1.11
- removed net N$6: U1.19
- removed net VSS: X1.10
- net GND: now also U1.11, U1.19, X1.10, X7.1
- net N$35: no longer C6.1
- net VCC: now also C6.1, R4.2, R6.2, X1.9
- net VDD: no longer R6.2, X1.9
Routing:
- net VDD: track 129.6 -> 15.4 mm, vias 0 -> 2
- net N$35: track 84.7 -> 7.39 mm
- net VCC: track 121.0 -> 174.4 mm
- net N$7: track 108.7 -> 68.6 mm
- net GND: track 256.7 -> 283.6 mm, vias 3 -> 2
- net N$27: track 36.9 -> 15.9 mm
- net N$22: track 32.9 -> 21.2 mm, vias 0 -> 1
- net N$16: track 85.8 -> 74.4 mm
- net N$12: track 84.9 -> 95.7 mm, vias 6 -> 2
- net N$1: track 35.5 -> 27.5 mm, vias 1 -> 0
- net N$10: track 37.3 -> 29.9 mm, vias 3 -> 2
- net N$2: track 31.1 -> 24.0 mm, vias 4 -> 2
- net N$18: track 34.0 -> 28.1 mm, vias 0 -> 2
- net N$33: track 50.1 -> 55.1 mm
- net N$23: track 26.0 -> 30.2 mm
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
Commit message: updates
Parts:
- X1: value 332-10 -> port c
- X2: value 332-10 -> analog I/O bus
- X3: value 332-10 -> port a
Changed lines of the file:
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@@
 <?xml version="1.0" encoding="utf-8"?>
 <!DOCTYPE eagle SYSTEM "eagle.dtd">
-<eagle version="7.5.0">
+<eagle version="7.6.0">
 <drawing>
 <settings>
@@
 <element name="U1" library="SparkFun-DigitalIC" package="DIL20" value="TPIC6B595PTH" x="20.32" y="71.12" rot="R270"/>
 <element name="U2" library="SparkFun-DigitalIC" package="DIL20" value="TPIC6B595PTH" x="31.75" y="71.12" rot="R270"/>
-<element name="X1" library="con-garry" package="332-10" value="332-10" x="66.04" y="55.88"/>
-<element name="X2" library="con-garry" package="332-10" value="332-10" x="68.58" y="68.58" rot="R270"/>
-<element name="X3" library="con-garry" package="332-10" value="332-10" x="64.77" y="83.82"/>
+<element name="X1" library="con-garry" package="332-10" value="port c" x="66.04" y="55.88"/>
+<element name="X2" library="con-garry" package="332-10" value="analog I/O bus" x="68.58" y="68.58" rot="R270"/>
+<element name="X3" library="con-garry" package="332-10" value="port a" x="64.77" y="83.82"/>
 <element name="X4" library="con-garry" package="332-10" value="332-10" x="45.72" y="55.88"/>
 <element name="DIS1" library="display-hp" package="HP5082" value="HP5082" x="44.45" y="76.2">
